File: eagle/teensy-dsc.sch (EAGLE design)
At the start: 27 parts, among them J1 RJ11-6PTH, J2 RJ11-6PTH, J3 RJ45-8PTH, J4 POWER_JACKPTH, M1 XBEERX-VN, Q1 IRLML6344, X1 STEREOJACK, X2 STEREOJACK

Commit message: Start v0.9 board design
- Has two 1x16 headers for expansion boards
- 85x55mm design
- four mounting holes
- ports on two sides
Parts:
- removed M1: XBEERX-VN, xbee_r1:XBEERX-VN
- removed OK1: LTV826S, optocoupler:LTV826S
- added J5: USB-B, SparkFun-Connectors:USBPTH
- added JP2: M16PTH, SparkFun-Connectors:M16PTH
- added U$5: XBEERX-VN, xbee_r1:XBEERX-VN
- added U$6: LTV826S, optocoupler:LTV826S
- C1: device SparkFun-Capacitors:1.0UF-25V-+80/-20(0805) -> rcl:C-EUC0805
- C2: device SparkFun-Capacitors:22UF-6.3V-20%(0805) -> rcl:C-EUC0805
- C3, C4, C5, C6, C7: device SparkFun-Passives:CAP0805 -> rcl:C-EUC0805
- JP1: value USB-B -> M16PTH; device SparkFun-Connectors:USBPTH -> SparkFun-Connectors:M16PTH
- R1, R2: device SparkFun-Resistors:0.75OHM1/4W1%(0805) -> resistor:R-US_M0805
- U$1: value TEENSY_3.1_BASIC -> TEENSY_3.1_ALL_PINS_AND_PADS; device Teensy_3_Series_Board_v1.0:TEENSY_3.1_BASIC -> Teensy_3_Series_Board_v1.0:TEENSY_3.1_ALL_PINS_AND_PADS
Connections:
- new net A10: JP2.8, U$1.A10
- new net A11: JP2.7, U$1.A11
- new net A12: JP2.6, U$1.A12
- new net A13: JP2.5, U$1.A13
- new net AGND: JP2.4, U$1.AGND
- new net AREF: JP2.3, U$1.AREF
- new net P11: JP1.14, U$1.11/MOSI
- new net P12: JP1.13, U$1.12/MISO
- new net P13: JP1.12, U$1.13/SCK/LED
- new net P14: JP1.11, U$1.14/A0
- new net P15: JP1.10, U$1.15/A1/T
- new net P16: JP1.9, U$1.16/A2/T
- new net P17: JP1.8, U$1.17/A3/T
- new net P18: JP1.7, U$1.18/A4/T/SDA0
- new net P19: JP1.6, U$1.19/A5/T/SCL0
- new net P2: JP1.15, U$1.2
- new net P24: JP1.5, U$1.24
- new net P25: JP1.3, U$1.25/T/PWM
- new net P26: JP1.4, U$1.26/A15
- new net P27: JP2.15, U$1.27/A16
- new net P28: JP2.14, U$1.28/A17
- new net P29: JP2.13, U$1.29/A18/SCL1
- new net P30: JP2.12, U$1.30/A19/SDA1
- new net P31: JP2.11, U$1.31/A20
- new net P32: JP2.10, U$1.32/T/PWM
- new net P33: JP2.9, U$1.33/T
- new net PGM: JP2.2, U$1.PGM
- net +12V: now also JP1.2
- net 3.3V: now also JP2.1, U$5.VCC@1; no longer M1.VCC@1
- net 5V: now also J5.VBUS, JP1.16; no longer JP1.VBUS
- net FOCUS: now also U$6A.COL; no longer OK1A.COL
- net FOCUS-CTL: now also U$6A.A; no longer OK1A.A
- net GND: now also J5.GND, JP1.1, U$5.GND@10; no longer JP1.GND, M1.GND@10
- net GND_MAIN: now also JP2.16
- net N$7: now also U$6B.C; no longer OK1B.C
- net N$9: now also U$6A.C; no longer OK1A.C
- net SHUTTER: now also U$6B.COL; no longer OK1B.COL
- net SHUTTER-CTL: now also U$6B.A; no longer OK1B.A
- net SHUTTER-GND: now also U$6A.EMIT, U$6B.EMIT; no longer OK1A.EMIT, OK1B.EMIT
- net XBEE_IN: now also U$5.DIN; no longer M1.DIN
- net XBEE_OUT: now also U$5.DOUT; no longer M1.DOUT
- net XBEE_RST: now also U$1.A14/DAC, U$5.RESET#; no longer M1.RESET#, U$1.2
Other:
- note removed: "Aaron Turner http://synfin.net/teensydsc"
- note removed: "v0.3"
- moved on the sheet: C1, C2, C3, C4, C5, C6, C7, C8, C9, D5, J1, J2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
